Commit message: Combined quad encoder and motors to work with diff drive controller

File: rocko_env/rocko_env/description/ros2_control/rocko.ros2_control.xacro (robot description, xacro)
@@ -7,8 +7,6 @@
         <param name="pinNumberSpeed">1</param>
         <param name="pinNumberDirection">2</param>
-        <param name="pinNumberAChannel">5</param>
-        <param name="pinNumberBChannel">6</param>
       </hardware>
-      <joint name="left_wheel_joint">
+      <joint name="left_wheel">
         <command_interface name="velocity"/>
         <state_interface name="position"/>
@@ -21,8 +19,6 @@
         <param name="pinNumberSpeed">3</param>
         <param name="pinNumberDirection">4</param>
-        <param name="pinNumberAChannel">7</param>
-        <param name="pinNumberBChannel">8</param>
       </hardware>
-      <joint name="right_wheel_joint">
+      <joint name="right_wheel">
         <command_interface name="velocity"/>
         <state_interface name="position"/>
@@ -40,5 +36,5 @@
       </sensor>
     </ros2_control>
-    <ros2_control name="LeftRelativeEncoder" type="sensor">
+    <!-- <ros2_control name="LeftRelativeEncoder" type="sensor">
       <hardware>
         <plugin>rocko_env/QuadEncoder</plugin>
@@ -57,5 +53,5 @@
         <state_interface name="velocity"/>
       </sensor>
-    </ros2_control>
+    </ros2_control> -->
   </xacro:macro>
 </robot>

Commit message: Tested controller without hardware

File: rocko_env/rocko_env/description/ros2_control/rocko.ros2_control.xacro (robot description, xacro)
@@ -8,5 +8,5 @@
         <param name="pinNumberDirection">2</param>
       </hardware>
-      <joint name="left_wheel">
+      <joint name="left_wheel_joint">
         <command_interface name="velocity"/>
         <state_interface name="position"/>
@@ -20,5 +20,5 @@
         <param name="pinNumberDirection">4</param>
       </hardware>
-      <joint name="right_wheel">
+      <joint name="right_wheel_joint">
         <command_interface name="velocity"/>
         <state_interface name="position"/>
@@ -36,22 +36,4 @@
       </sensor>
     </ros2_control>
-    <!-- <ros2_control name="LeftRelativeEncoder" type="sensor">
-      <hardware>
-        <plugin>rocko_env/QuadEncoder</plugin>
-      </hardware>
-      <sensor name="left_quad_encoder">
-        <state_interface name="position"/>
-        <state_interface name="velocity"/>
-      </sensor>
-    </ros2_control>
-    <ros2_control name="RightRelativeEncoder" type="sensor">
-      <hardware>
-        <plugin>rocko_env/QuadEncoder</plugin>
-      </hardware>
-      <sensor name="right_quad_encoder">
-        <state_interface name="position"/>
-        <state_interface name="velocity"/>
-      </sensor>
-    </ros2_control> -->
   </xacro:macro>
 </robot>

Commit message: It's messy, but the PID does output to motors

File: rocko_env/rocko_env/description/ros2_control/rocko.ros2_control.xacro (robot description, xacro)
@@ -30,9 +30,19 @@
         <plugin>rocko_env/ICM20948</plugin>
       </hardware>
-      <sensor name="icm20948">
+      <!-- <sensor name="icm20948">
         <state_interface name="yaw"/>
         <state_interface name="pitch"/>
         <state_interface name="roll"/>
-      </sensor>
+      </sensor> -->
+      <joint name="left_wheel_joint">
+        <state_interface name="yaw"/>
+        <state_interface name="pitch"/>
+        <state_interface name="roll"/>
+      </joint>
+      <joint name="right_wheel_joint">
+        <state_interface name="yaw"/>
+        <state_interface name="pitch"/>
+        <state_interface name="roll"/>
+      </joint>
     </ros2_control>
   </xacro:macro>
