Commit message: Make use_mock_hardware real and let rocko_env build off the Pi
use_mock_hardware was accepted by the launch files and the xacro and then
ignored (and two launch files defaulted it to "true"), and rocko_env could not
be built anywhere but a Raspberry Pi because the motor plugin needs WiringPi.
This is ADR 0003 follow-ons 1 and 2.

- xacro: use_mock_hardware:=true selects one mock_components/GenericSystem
  block ("MockRocko") with the same joints and interface names as the real
  hardware, so rocko_controllers.yaml loads against it unchanged. The real
  <ros2_control> blocks are untouched (their expanded XML is identical to
  before). The mock has no physics: it is a wiring check, not a simulation.
- launch: use_mock_hardware now defaults to false in all three launch files
  (it was "true" in two, which would have swapped the real motors for a mock
  once the flag worked). The IMU and encoder nodes are skipped under the mock,
  a MOCK HARDWARE banner is printed, and the URDF is passed as a string
  parameter so a ": " in an xacro comment cannot break the launch.
- CMake: ROCKO_SKIP_WIRINGPI leaves out the motor plugin. The default is
  unchanged and still requires WiringPi; skipping where WiringPi exists is an
  error, because CMake caches the option and a stale ON would build a robot
  without its motor driver.
- build_ros.sh always passes the flag, compose sets it to ON, and a failed
  build now exits 1 instead of printing Done! and exiting 0.
- package.xml: declare pid_controller and diff_drive_controller, which the
  launch files already needed.
- Five Python executables get the executable bit; they were 100644, so
  --symlink-install could not run them.
- verify_urdf.sh (Tier 0) and verify_mock.sh (Tier 2): expand every mode and
  assert what is in it, compare the mock's interfaces with the real hardware's,
  and bring the controllers up against the mock. Each was shown to fail on a
  deliberate break.

Verified in the dev container (ros:jazzy, arm64): build_ros.sh exits 0 and
exits 1 on a forced failure; verify_urdf.sh and verify_mock.sh (balance and
tank) pass; their negative controls fail for the right reason. Not verified:
anything on a Raspberry Pi. Motor12VoltQuadEncoder.cpp is not compiled off a
Pi, and the mock says nothing about whether the robot balances.

Co-Authored-By: Claude Sonnet 5.5 <noreply@anthropic.com>

File: rocko_env/rocko_env/description/ros2_control/rocko.ros2_control.xacro (robot description, xacro)
@@ -2,4 +2,39 @@
 <robot xmlns:xacro="http://www.ros.org/wiki/xacro">
   <xacro:macro name="rocko_ros2_control" params="name prefix use_mock_hardware">
+    <!-- use_mock_hardware:=true  -> the one MockRocko system below.
+         use_mock_hardware:=false -> the real motor and IMU plugins (what runs on the robot). -->
+    <xacro:if value="${use_mock_hardware}">
+      <!-- A WIRING CHECK, NOT A SIMULATION. mock_components/GenericSystem has no physics: it
+           echoes each velocity command back as that joint's velocity state, and the IMU states
+           (yaw/pitch/roll) stay at 0.0. A balance controller therefore always looks "fine" here.
+           What it does prove: every controller rocko.launch.py spawns (the four cascade
+           controllers) loads, claims interfaces that exist, and chains and activates.
+           It exports the same joint and interface names as the real plugins, so the real
+           rocko_controllers.yaml loads against it unchanged. Keep the two in step. -->
+      <ros2_control name="MockRocko" type="system">
+        <hardware>
+          <plugin>mock_components/GenericSystem</plugin>
+        </hardware>
+        <joint name="left_wheel_joint">
+          <command_interface name="velocity"/>
+          <state_interface name="position"/>
+          <state_interface name="velocity"/>
+          <state_interface name="yaw"/>
+          <state_interface name="pitch"/>
+          <state_interface name="roll"/>
+        </joint>
+        <joint name="right_wheel_joint">
+          <command_interface name="velocity"/>
+          <state_interface name="position"/>
+          <state_interface name="velocity"/>
+          <state_interface name="yaw"/>
+          <state_interface name="pitch"/>
+          <state_interface name="roll"/>
+        </joint>
+      </ros2_control>
+    </xacro:if>
+    <!-- The real hardware, exactly as it was before the mock existed. Not re-indented, so the
+         diff shows that nothing inside changed. -->
+    <xacro:unless value="${use_mock_hardware}">
     <ros2_control name="LeftDriveMotor" type="actuator">
       <hardware>
@@ -48,4 +83,5 @@
       </joint>
     </ros2_control>
+    </xacro:unless>
   </xacro:macro>
 </robot>

File: rocko_env/rocko_env/description/ros2_control/rocko_tank_mode.ros2_control.xacro (robot description, xacro)
@@ -2,4 +2,29 @@
 <robot xmlns:xacro="http://www.ros.org/wiki/xacro">
   <xacro:macro name="rocko_ros2_control" params="name prefix use_mock_hardware">
+    <!-- use_mock_hardware:=true  -> the one MockRocko system below.
+         use_mock_hardware:=false -> the real motor plugins (what runs on the robot). -->
+    <xacro:if value="${use_mock_hardware}">
+      <!-- A WIRING CHECK, NOT A SIMULATION: no physics, each velocity command is echoed back as
+           that joint's velocity state. Same joint and interface names as the real plugins, so
+           rocko_tank_mode_controllers.yaml loads against it unchanged. -->
+      <ros2_control name="MockRocko" type="system">
+        <hardware>
+          <plugin>mock_components/GenericSystem</plugin>
+        </hardware>
+        <joint name="left_wheel_joint">
+          <command_interface name="velocity"/>
+          <state_interface name="position"/>
+          <state_interface name="velocity"/>
+        </joint>
+        <joint name="right_wheel_joint">
+          <command_interface name="velocity"/>
+          <state_interface name="position"/>
+          <state_interface name="velocity"/>
+        </joint>
+      </ros2_control>
+    </xacro:if>
+    <!-- The real hardware, exactly as it was before the mock existed. Not re-indented, so the
+         diff shows that nothing inside changed. -->
+    <xacro:unless value="${use_mock_hardware}">
     <ros2_control name="LeftDriveMotor" type="actuator">
       <hardware>
@@ -28,4 +53,5 @@
       </joint>
     </ros2_control>
+    </xacro:unless>
   </xacro:macro>
 </robot>
